Commit message: window update using local bellan recursion

File: experiments/Go2_sim_kunzhao/descriptions/urdf/go2.urdf (robot description, URDF)
Before this commit: robot go2_description, 42 links, 41 joints
Links:
- link FL_calf: mass 0.154 -> 0.241352; geometry collision cylinder length=0.12 radius=0.012; visual mesh filename=experiments/Go2_sim_kunzhao/descriptions/meshes/calf_0.obj
- link FL_calf_rotor: mass 0.001 -> 0.089
- link FL_foot: mass 0.04 -> 0.06; geometry collision sphere radius=0.022; visual mesh filename=experiments/Go2_sim_kunzhao/descriptions/meshes/foot.obj
- link FL_hip: geometry collision cylinder length=0.04 radius=0.046; visual mesh filename=experiments/Go2_sim_kunzhao/descriptions/meshes/hip_0.obj
- link FL_hip_rotor: mass 0.001 -> 0.089
- link FL_thigh: geometry collision box size=0.213 0.0245 0.034; visual mesh filename=experiments/Go2_sim_kunzhao/descriptions/meshes/thigh_0.obj
- link FL_thigh_rotor: mass 0.001 -> 0.089
- link FR_calf: mass 0.154 -> 0.241352; geometry collision cylinder length=0.12 radius=0.013; visual mesh filename=experiments/Go2_sim_kunzhao/descriptions/meshes/calf_mirror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
- link FR_calf_rotor: mass 0.001 -> 0.089
- link FR_foot: mass 0.04 -> 0.06; geometry collision sphere radius=0.022; visual mesh filename=experiments/Go2_sim_kunzhao/descriptions/meshes/foot.obj
- link FR_hip: geometry collision cylinder length=0.04 radius=0.046; visual mesh filename=experiments/Go2_sim_kunzhao/descriptions/meshes/hip_0.obj
- link FR_hip_rotor: mass 0.001 -> 0.089
- link FR_thigh: geometry collision box size=0.213 0.0245 0.034; visual mesh filename=experiments/Go2_sim_kunzhao/descriptions/meshes/thigh_mirro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
- link FR_thigh_rotor: mass 0.001 -> 0.089
- link Head_lower: mass 0.001 -> None
- link Head_upper: mass 0.001 -> None
- link RL_calf: mass 0.154 -> 0.241352; geometry collision cylinder length=0.12 radius=0.013; visual mesh filename=experiments/Go2_sim_kunzhao/descriptions/meshes/calf_0.obj
- link RL_calf_rotor: mass 0.001 -> 0.089
- link RL_foot: mass 0.04 -> 0.06; geometry collision sphere radius=0.022; visual mesh filename=experiments/Go2_sim_kunzhao/descriptions/meshes/foot.obj
- link RL_hip: geometry collision cylinder length=0.04 radius=0.046; visual mesh filename=experiments/Go2_sim_kunzhao/descriptions/meshes/hip_0.obj
- link RL_hip_rotor: mass 0.001 -> 0.089
- link RL_thigh: geometry collision box size=0.213 0.0245 0.034; visual mesh filename=experiments/Go2_sim_kunzhao/descriptions/meshes/thigh_0.obj
- link RL_thigh_rotor: mass 0.001 -> 0.089
- link RR_calf: mass 0.154 -> 0.241352; geometry collision cylinder length=0.12 radius=0.013; visual mesh filename=experiments/Go2_sim_kunzhao/descriptions/meshes/calf_mirror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
- link RR_calf_rotor: mass 0.001 -> 0.089
- link RR_foot: mass 0.04 -> 0.06; geometry collision sphere radius=0.022; visual mesh filename=experiments/Go2_sim_kunzhao/descriptions/meshes/foot.obj
- link RR_hip: geometry collision cylinder length=0.04 radius=0.046; visual mesh filename=experiments/Go2_sim_kunzhao/descriptions/meshes/hip_0.obj
- link RR_hip_rotor: mass 0.001 -> 0.089
- link RR_thigh: geometry collision box size=0.213 0.0245 0.034; visual mesh filename=experiments/Go2_sim_kunzhao/descriptions/meshes/thigh_mirro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
- link RR_thigh_rotor: mass 0.001 -> 0.089
- link base: geometry collision box size=0.3762 0.0935 0.114; visual mesh filename=experiments/Go2_sim_kunzhao/descriptions/meshes/base_0.obj
